Commit message: psuhing working multiobj

File: roboverse/envs/assets/sawyer_robot/sawyer_description/urdf/sawyer_xacro_finger_visual_only.urdf (robot description, URDF)
Before this commit: robot sawyer, 27 links, 26 joints
Links:
- link pedestal: geometry collision cylinder length=0.62 radius=0.18; visual cylinder length=0.62 radius=0.18
- link right_arm_base_link: geometry collision cylinder length=0.24 radius=0.08; visual cylinder length=0.24 radius=0.08
- link right_l0: geometry collision sphere radius=0.07; visual sphere radius=0.07
- link right_l1: geometry collision sphere radius=0.07; visual sphere radius=0.07
- link right_l2: geometry collision cylinder length=0.35 radius=0.06; visual cylinder length=0.35 radius=0.06
- link right_l3: geometry collision sphere radius=0.06; visual sphere radius=0.06
- link right_l4: geometry collision cylinder length=0.36 radius=0.045; visual cylinder length=0.36 radius=0.045
